File: ibScaleFeederLite.kicad_pcb (KiCad board)
At the start: 4 copper layers, 51.6 x 89 mm, 89 parts, among them J1 PEEL, J2 DRIVE, J3 RAIL, J4 SWD, J5 Serial, J6 SWD, SW1 DOWN, SW2 UP, SW3 BOOT, U2 DRV8837, U3 DRV8837, U4 THVD1400D, U5 TPS563300, U6 AMS1117-3.3, U9 STM32F031C6Tx, Y1 8MHz

Commit message: update L1 to use correct VLX4045EX footprint instead of generic one
Parts:
- L1: footprint Inductor_SMD:L_6.3x6.3_H3 -> Inductor_SMD:L_TDK_VLS6045EX_VLS6045AF
Changed lines of the file:
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@@
 		(tags "WSON 8 1EP ThermalVias")
 		(property "Reference" "U2"
-			(at 2.371 0.5878 270)
+			(at 2.621 -0.0122 0)
 			(layer "F.SilkS")
 			(effects
@@
 		(tags "capacitor handsolder")
 		(property "Reference" "C9"
-			(at 2.5654 0 0)
+			(at 2.6585 0 0)
 			(layer "F.SilkS")
 			(effects
@@
 		)
 	)
-	(footprint "Inductor_SMD:L_6.3x6.3_H3"
+	(footprint "Inductor_SMD:L_TDK_VLS6045EX_VLS6045AF"
 		(layer "F.Cu")
 		(at 130.317423 42.179234 -90)
-		(descr "Choke, SMD, 6.3x6.3mm 3mm height")
-		(tags "Choke SMD")
+		(descr "Inductor,TDK, VLS-6045, 6x6x4.5mm, https://product.tdk.com/system/files/dam/doc/product/inductor/inductor/smd/catalog/inductor_commercial_power_vls6045ex_en.pdf")
+		(tags "inductor TDK VLS SMD VLS6045EF VLS6045AF")
 		(property "Reference" "L1"
-			(at -4.222984 -0.026327 0)
+			(at 0 -4 270)
+			(unlocked yes)
 			(layer "F.SilkS")
 			(effects
@@
 		)
 		(property "Value" "10uh"
-			(at 0 4.45 90)
+			(at 0 4 270)
+			(unlocked yes)
 			(layer "F.Fab")
 			(effects
@@
 		(duplicate_pad_numbers_are_jumpers no)
 		(fp_line
-			(start -3.3 3.2)
-			(end -3.3 1.5)
+			(start -3.1 3.1)
+			(end 3.1 3.1)
 			(stroke
 				(width 0.12)
@@
 		)
 		(fp_line
-			(start 3.3 3.2)
-			(end -3.3 3.2)
+			(start -3.1 3.1)
+			(end -3.1 2.7)
 			(stroke
 				(width 0.12)
@@
 		)
 		(fp_line
-			(start 3.3 1.5)
-			(end 3.3 3.2)
+			(start 3.1 3.1)
+			(end 3.1 2.7)
 			(stroke
 				(width 0.12)
@@
 		)
 		(fp_line
-			(start -3.3 -1.5)
-			(end -3.3 -3.2)
+			(start -3.1 -3.1)
+			(end -3.1 -2.7)
 			(stroke
 				(width 0.12)
@@
 		)
 		(fp_line
-			(start -3.3 -3.2)
-			(end 3.3 -3.2)
+			(start -3.1 -3.1)
+			(end 3.1 -3.1)
 			(stroke
 				(width 0.12)
@@
 		)
 		(fp_line
-			(start 3.3 -3.2)
-			(end 3.3 -1.5)
+			(start 3.1 -3.1)
+			(end 3.1 -2.7)
 			(stroke
 				(width 0.12)
@@
 			(layer "F.SilkS")
 		)
-		(fp_line
-			(start -3.75 3.4)
-			(end 3.75 3.4)
-			(stroke
-				(width 0.05)
-				(type solid)
-			)
-			(layer "F.CrtYd")
-		)
-		(fp_line
-			(start 3.75 3.4)
-			(end 3.75 -3.4)
-			(stroke
-				(width 0.05)
-				(type solid)
-			)
-			(layer "F.CrtYd")
-		)
-		(fp_line
-			(start -3.75 -3.4)
-			(end -3.75 3.4)
-			(stroke
-				(width 0.05)
-				(type solid)
-			)
-			(layer "F.CrtYd")
-		)
-		(fp_line
-			(start 3.75 -3.4)
-			(end -3.75 -3.4)
+		(fp_rect
+			(start -3.3 -3.25)
+			(end 3.3 3.25)
 			(stroke
 				(width 0.05)
 				(type solid)
 			)
+			(fill no)
 			(layer "F.CrtYd")
 		)
-		(fp_line
-			(start -3.15 3.15)
-			(end 3.15 3.15)
-			(stroke
-				(width 0.1)
-				(type solid)
-			)
-			(layer "F.Fab")
-		)
-		(fp_line
-			(start -3.15 3.15)
-			(end -3.15 1.5)
-			(stroke
-				(width 0.1)
-				(type solid)
-			)
-			(layer "F.Fab")
-		)
-		(fp_line
-			(start 3.15 3.15)
-			(end 3.15 1.5)
-			(stroke
-				(width 0.1)
-				(type solid)
-			)
-			(layer "F.Fab")
-		)
-		(fp_line
-			(start -3.15 -3.15)
-			(end -3.15 -1.5)
-			(stroke
-				(width 0.1)
-				(type solid)
-			)
-			(layer "F.Fab")
-		)
-		(fp_line
-			(start -3.15 -3.15)
-			(end 3.15 -3.15)
-			(stroke
-				(width 0.1)
-				(type solid)
-			)
-			(layer "F.Fab")
-		)
-		(fp_line
-			(start 3.15 -3.15)
-			(end 3.15 -1.5)
-			(stroke
-				(width 0.1)
-				(type solid)
-			)
-			(layer "F.Fab")
-		)
-		(fp_arc
-			(start 1.91 1.91)
-			(mid 0 2.701148)
-			(end -1.91 1.91)
-			(stroke
-				(width 0.1)
-				(type solid)
-			)
-			(layer "F.Fab")
-		)
-		(fp_arc
-			(start -1.91 -1.91)
-			(mid 0 -2.701148)
-			(end 1.91 -1.91)
+		(fp_rect
+			(start -3 -3)
+			(end 3 3)
 			(stroke
 				(width 0.1)
 				(type solid)
 			)
+			(fill no)
 			(layer "F.Fab")
 		)
 		(fp_text user "${REFERENCE}"
-			(at 0 0 90)
+			(at 0 0 270)
+			(unlocked yes)
 			(layer "F.Fab")
 			(effects
@@
 			)
 		)
-		(pad "1" smd rect
-			(at -2.75 0 270)
-			(size 1.5 2.4)
+		(pad "1" smd roundrect
+			(at -2.1 0 270)
+			(size 1.9 5.1)
 			(layers "F.Cu" "F.Mask" "F.Paste")
+			(roundrect_rratio 0.25)
 			(net "Net-(U5-SW)")
 			(pintype "passive")
 		)
-		(pad "2" smd rect
-			(at 2.75 0 270)
-			(size 1.5 2.4)
+		(pad "2" smd roundrect
+			(at 2.1 0 270)
+			(size 1.9 5.1)
 			(layers "F.Cu" "F.Mask" "F.Paste")
+			(roundrect_rratio 0.25)
 			(net "+10V")
 			(pintype "passive")
 		)
 		(embedded_fonts no)
-		(model "${KICAD10_3DMODEL_DIR}/Inductor_SMD.3dshapes/L_Sunlord_SWPA6040S.step"
+		(model "${KICAD10_3DMODEL_DIR}/Inductor_SMD.3dshapes/L_TDK_VLS6045EX_VLS6045AF.step"
 			(offset
 				(xyz 0 0 0)
@@
 		(tags "capacitor handsolder")
 		(property "Reference" "C5"
-			(at -2.5654 0 0)
+			(at 2.6625 0 0)
 			(layer "F.SilkS")
 			(effects
@@
 	)
 	(gr_text "PEEL"
-		(at 112.419869 63.857914 0)
+		(at 112.5 62.15 0)
 		(layer "F.SilkS")
 		(effects
